File: PCB/project.sch (KiCad schematic (older format))
At the start: 98 parts, among them IC1 ATTINY2313-P, J1 AVR-ISP-6, P1 CONN_1, P13 CONN_1, P14 CONN_1, P15 CONN_1, P16 CONN_1, P17 CONN_1, P18 CONN_1, P19 CONN_1, P2 CONN_1, P20 CONN_1, P21 CONN_1, P22 CONN_1, P23 CONN_1, P24 CONN_1, P25 CONN_1, P27 CONN_1, P28 CONN_1, P3 MIDI_IN, P31 CONN_1, P36 CONN_1, P37 CONN_1, P38 CONN_1, P4 MIDI_THRU, P40 CONN_1, P41 CONN_1, P42 CONN_1, P43 CONN_1, P44 CONN_1, P46 CONN_1, U1 TLC274, U10 TL082, U11 TL082, U2 LT1054, U3 4051, U4 7805, U5 7809, U6 7909, U7 4051, U9 DAC0808, X1 CRYSTAL

Commit message: cleaned up a bit
Parts:
- C15, C16: value 22n -> 22p
- X1: value CRYSTAL -> 12MHz
Connections:
- wire segments 174 -> 186
Other:
- moved on the sheet: J1
Changed lines of the file:
@@
-EESchema Schematic File Version 2  date Mi 28 Dez 2011 02:52:30 CET
+EESchema Schematic File Version 2  date So 27 Jul 2014 13:20:00 CEST
 LIBS:power
-LIBS:device
-LIBS:transistors
-LIBS:conn
-LIBS:linear
-LIBS:regul
-LIBS:74xx
-LIBS:cmos4000
-LIBS:adc-dac
-LIBS:memory
-LIBS:xilinx
-LIBS:special
-LIBS:microcontrollers
-LIBS:dsp
-LIBS:microchip
-LIBS:analog_switches
-LIBS:motorola
-LIBS:texas
-LIBS:intel
-LIBS:audio
-LIBS:interface
-LIBS:digital-audio
-LIBS:philips
-LIBS:display
-LIBS:cypress
-LIBS:siliconi
-LIBS:opto
-LIBS:atmel
-LIBS:contrib
-LIBS:valves
-LIBS:micha_custom
 LIBS:project-cache
-EELAYER 24  0
+EELAYER 25  0
 EELAYER END
 $Descr A4 11700 8267
+encoding utf-8
 Sheet 1 1
 Title ""
-Date "28 dec 2011"
+Date "27 jul 2014"
 Rev ""
 Comp ""
@@
 Comment4 ""
 $EndDescr
-Text Label 10750 6700 0    60   ~ 0
--9V
-Text Label 10300 6700 0    60   ~ 0
-+9V
-Text Label 9800 6700 0    60   ~ 0
-vcc
-Text Label 9300 6700 0    60   ~ 0
-gnd
+Connection ~ 5150 1450
+Wire Wire Line
+	5150 1600 5150 1300
+Wire Wire Line
+	8450 2600 8650 2600
+Wire Wire Line
+	8200 2350 8400 2350
+Wire Wire Line
+	8650 4950 8650 4650
+Connection ~ 8000 4600
+Wire Wire Line
+	8000 4800 8000 4550
+Wire Wire Line
+	3800 4800 4150 4800
+Wire Wire Line
+	3800 5000 4150 5000
+Wire Wire Line
+	4800 4900 4450 4900
 Connection ~ 10200 6400
 Connection ~ 10200 6200
@@
 	5800 1050 6100 1050
 Wire Wire Line
-	5150 1300 5150 1450
-Wire Wire Line
-	5150 650  5150 800
+	5150 800  5150 650
 Wire Notes Line
 	7400 500  11200 500
@@
 Wire Wire Line
 	9100 3200 9100 3450
-Wire Wire Line
-	8000 4550 8000 4600
 Wire Wire Line
 	8650 3850 8900 3850
@@
 	900  6250 1150 6250
 Wire Wire Line
-	800  7150 1150 7150
+	1150 7150 800  7150
 Wire Wire Line
 	1050 7350 1150 7350
@@
 Connection ~ 10200 6100
 Connection ~ 10200 6300
+Wire Wire Line
+	4450 4800 4800 4800
+Wire Wire Line
+	4450 5000 4800 5000
+Wire Wire Line
+	3800 4900 4150 4900
+Wire Wire Line
+	800  7150 800  7650
+Wire Wire Line
+	7700 2350 7500 2350
+Wire Wire Line
+	5150 650  5650 650
+Text Label 10750 6700 0    60   ~ 0
+-9V
+Text Label 10300 6700 0    60   ~ 0
++9V
+Text Label 9800 6700 0    60   ~ 0
+vcc
+Text Label 9300 6700 0    60   ~ 0
+gnd
 $Comp
 L CONN_1 P46
@@
 	0    1    1    0
 $EndComp
-Text Label 8650 2600 2    60   ~ 0
+Text Label 8450 2600 0    60   ~ 0
 gnd
 $Comp
@@
 Text Label 7950 1450 2    60   ~ 0
 portamento
-Text Label 7700 2350 2    60   ~ 0
+Text Label 7500 2350 0    60   ~ 0
 +9V
-Text Label 8200 2350 0    60   ~ 0
+Text Label 8400 2350 2    60   ~ 0
 -9V
 $Comp
@@
 	0    1    1    0
 $EndComp
-Text Label 8650 4650 3    60   ~ 0
+Text Label 8650 4800 3    60   ~ 0
 gnd
 $Comp
@@
 Text Label 7300 4050 2    60   ~ 0
 gnd
-Text Label 8000 4600 3    60   ~ 0
+Text Label 8000 4800 1    60   ~ 0
 -9V
 $Comp
@@
 P 6400 5150
 F 0 "C16" H 6450 5250 50  0000 L CNN
-F 1 "22n" H 6450 5050 50  0000 L CNN
+F 1 "22p" H 6450 5050 50  0000 L CNN
 	1    6400 5150
 	0    1    1    0
@@
 P 6400 4800
 F 0 "C15" H 6450 4900 50  0000 L CNN
-F 1 "22n" H 6450 4700 50  0000 L CNN
+F 1 "22p" H 6450 4700 50  0000 L CNN
 	1    6400 4800
 	0    1    1    0
@@
 P 5800 4950
 F 0 "X1" H 5800 5100 60  0000 C CNN
-F 1 "CRYSTAL" H 5800 4800 60  0000 C CNN
+F 1 "12MHz" H 5800 4800 60  0000 C CNN
 	1    5800 4950
 	0    1    1    0
@@
 Text Label 5800 2900 2    60   ~ 0
 vcc
-Text Label 4050 4800 2    60   ~ 0
+Text Label 3800 4800 2    60   ~ 0
 miso
-Text Label 4050 4900 2    60   ~ 0
+Text Label 3800 4900 2    60   ~ 0
 sck
-Text Label 4050 5000 2    60   ~ 0
+Text Label 3800 5000 2    60   ~ 0
 rst
-Text Label 4350 5000 0    60   ~ 0
-gnd
-Text Label 4350 4900 0    60   ~ 0
+Text Label 4800 5000 0    60   ~ 0
+gnd
+Text Label 4800 4900 0    60   ~ 0
 mosi
-Text Label 4350 4800 0    60   ~ 0
+Text Label 4800 4800 0    60   ~ 0
 vcc
 $Comp
 L AVR-ISP-6 J1
 U 1 1 4E8ADCE3
-P 4200 4900
-F 0 "J1" H 4050 5150 50  0000 C CNN
-F 1 "AVR-ISP-6" H 3950 4625 50  0000 L BNN
-F 2 "AVR-ISP-6" V 3700 4900 50  0001 C CNN
-	1    4200 4900
-	1    0    0    -1
-$EndComp
+P 4300 4900
+F 0 "J1" H 4150 5150 50  0000 C CNN
+F 1 "AVR-ISP-6" H 4050 4625 50  0000 L BNN
+F 2 "AVR-ISP-6" V 3800 4900 50  0001 C CNN
+	1    4300 4900
+	1    0    0    -1
+$EndComp
